File: clock.kicad_sch (KiCad schematic)
At the start: 7 parts

Commit message: moved to 6 layers, fixing DRC issues
Parts:
- added C34: 0402,100nF,50V,X7R, Capacitor_SMD:C_0402_1005Metric, symbol jlcpcb-basic-capacitor:0402,100nF,50V,X7R
- added R3: 10k, Resistor_SMD:R_0402_1005Metric, symbol jlcpcb-basic-resistor-0402:10k
- added X1: SIT9121AI-2C1-33E100.000000, my_lib:OSC-SMD_6P-L5.0-W3.2-BL-A, symbol my_lib:SIT9121AI-2C1-33E100.000000
- OSC1, OSC2, OSC3: now not fitted
Connections:
- net GND: now also C34.2, R3.2, X1.3 (GND)
- new net JX2_HD_SE_05_GC_N: X1.5 (OUT-)
- new net JX2_HD_SE_05_GC_P: X1.4 (OUT+)
- new net JX2_HD_SE_11_N: R3.1, X1.1 (OE/~{ST})
- new net VCCO_HD_26: C34.1, X1.6 (VDD)
