File: untitled.kicad_sch (KiCad schematic)
At the start: 44 parts, among them IC2 RT9187CGB, J7 PJ-002BH-SMT-TR, U5 AP62150WU, U6 AP62150WU, U8 AP62150WU, U9 AP62150WU

Commit message: moved jtag connector, added holes for all power supplies, fixed most of DRC
Parts:
- added J19: Conn_01x02_Pin, Connector_PinHeader_2.54mm:PinHeader_1x02_P2.54mm_Vertical, symbol Connector:Conn_01x02_Pin
- J7: now not fitted
- R18: value 10.5k -> 680; symbol jlcpcb-basic-resistor-0603:12k -> jlcpcb-basic-resistor-0603:680; LCSC C22790 -> C23228; MFGPN 0603WAF1202T5E -> 0603WAF6800T5E
- R22: LCSC C22790 -> C23046
Connections:
- net GND: now also J19.1 (Pin_1)
- net VIN_PIN: now also J19.2 (Pin_2)
Changed lines of the file:
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@@
 	)
 	(junction
+		(at 182.88 33.02)
+		(diameter 0)
+		(color 0 0 0 0)
+	)
+	(junction
 		(at 26.67 114.3)
 		(diameter 0)
@@
 	)
 	(junction
+		(at 185.42 30.48)
+		(diameter 0)
+		(color 0 0 0 0)
+	)
+	(junction
 		(at 110.49 171.45)
 		(diameter 0)
@@
 	(wire
 		(pts
+			(xy 182.88 33.02) (xy 187.96 33.02)
+		)
+		(stroke
+			(width 0)
+			(type default)
+		)
+	)
+	(wire
+		(pts
 			(xy 214.63 63.5) (xy 222.25 63.5)
 		)
@@
 	(wire
 		(pts
+			(xy 185.42 30.48) (xy 187.96 30.48)
+		)
+		(stroke
+			(width 0)
+			(type default)
+		)
+	)
+	(wire
+		(pts
 			(xy 251.46 71.12) (xy 251.46 73.66)
 		)
@@
 		(in_bom yes)
 		(on_board yes)
-		(dnp no)
+		(dnp yes)
 		(fields_autoplaced yes)
 		(property "Reference" "J7"
@@
 	)
 	(symbol
-		(lib_id "jlcpcb-basic-resistor-0603:12k")
+		(lib_id "jlcpcb-basic-resistor-0603:680")
 		(at 251.46 110.49 0)
 		(unit 1)
@@
 			)
 		)
-		(property "Value" "10.5k"
-			(at 245.872 113.284 0)
+		(property "Value" "680"
+			(at 246.634 111.252 0)
 			(effects
 				(font
@@
 			)
 		)
-		(property "Datasheet" "https://datasheet.lcsc.com/lcsc/2110252030_UNI-ROYAL-Uniroyal-Elec-0603WAF1202T5E_C22790.pdf"
+		(property "Datasheet" "https://datasheet.lcsc.com/lcsc/2110252130_UNI-ROYAL-Uniroyal-Elec-0603WAF6800T5E_C23228.pdf"
 			(at 251.46 110.49 0)
 			(effects
@@
 			)
 		)
-		(property "Description" "1% 1 10W Thick Film Resistors 75V   100ppm    -55    155   12k   0603 Chip Resistor - Surface Mount ROHS"
+		(property "Description" "1% 1 10W Thick Film Resistors 75V   100ppm    -55    155   680   0603 Chip Resistor - Surface Mount ROHS"
 			(at 251.46 110.49 0)
 			(effects
@@
 			)
 		)
-		(property "LCSC" "C22790"
+		(property "LCSC" "C23228"
 			(at 251.46 110.49 0)
 			(effects
@@
 			)
 		)
-		(property "MFGPN" "0603WAF1202T5E"
+		(property "MFGPN" "0603WAF6800T5E"
 			(at 251.46 110.49 0)
 			(effects
@@
 	)
 	(symbol
+		(lib_id "Connector:Conn_01x02_Pin")
+		(at 193.04 33.02 180)
+		(unit 1)
+		(exclude_from_sim no)
+		(in_bom yes)
+		(on_board yes)
+		(dnp yes)
+		(fields_autoplaced yes)
+		(property "Reference" "J19"
+			(at 194.31 30.4799 0)
+			(effects
+				(font
+					(size 1.27 1.27)
+				)
+				(justify right)
+			)
+		)
+		(property "Value" "Conn_01x02_Pin"
+			(at 194.31 33.0199 0)
+			(effects
+				(font
+					(size 1.27 1.27)
+				)
+				(justify right)
+				(hide yes)
+			)
+		)
+		(property "Footprint" "Connector_PinHeader_2.54mm:PinHeader_1x02_P2.54mm_Vertical"
+			(at 193.04 33.02 0)
+			(effects
+				(font
+					(size 1.27 1.27)
+				)
+				(hide yes)
+			)
+		)
+		(property "Datasheet" "~"
+			(at 193.04 33.02 0)
+			(effects
+				(font
+					(size 1.27 1.27)
+				)
+				(hide yes)
+			)
+		)
+		(property "Description" "Generic connector, single row, 01x02, script generated"
+			(at 193.04 33.02 0)
+			(effects
+				(font
+					(size 1.27 1.27)
+				)
+				(hide yes)
+			)
+		)
+		(pin "2"
+		)
+		(pin "1"
+		)
+		(instances
+			(project ""
+				(path "/72db9dae-5f31-4a10-9047-fdf9bc345a06/1803d24e-9660-4c9d-82db-3dd492b14553"
+					(reference "J19")
+					(unit 1)
+				)
+			)
+		)
+	)
+	(symbol
 		(lib_id "power:GND")
 		(at 251.46 128.27 0)
@@
 			)
 		)
-		(property "LCSC" "C22790"
+		(property "LCSC" "C23046"
 			(at 110.49 166.37 0)
 			(effects

Commit message: fixed jtag vref was not connected to 1.8V
Connections:
- net MGTRAVTT renamed +1V8
Changed lines of the file:
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@@
 	(paper "A4")
 	(junction
+		(at 254 60.96)
+		(diameter 0)
+		(color 0 0 0 0)
+	)
+	(junction
 		(at 266.7 105.41)
 		(diameter 0)
@@
 	(wire
 		(pts
+			(xy 254 60.96) (xy 261.62 60.96)
+		)
+		(stroke
+			(width 0)
+			(type default)
+		)
+	)
+	(wire
+		(pts
 			(xy 26.67 110.49) (xy 26.67 114.3)
 		)
@@
 	(wire
 		(pts
-			(xy 251.46 60.96) (xy 261.62 60.96)
+			(xy 251.46 60.96) (xy 254 60.96)
 		)
 		(stroke
@@
 	(wire
 		(pts
+			(xy 254 55.88) (xy 254 60.96)
+		)
+		(stroke
+			(width 0)
+			(type default)
+		)
+	)
+	(wire
+		(pts
 			(xy 115.57 68.58) (xy 115.57 71.12)
 		)
@@
 					(unit 1)
 				)
+			)
+		)
+	)
+	(symbol
+		(lib_id "power:+1V8")
+		(at 254 55.88 0)
+		(unit 1)
+		(exclude_from_sim no)
+		(in_bom yes)
+		(on_board yes)
+		(dnp no)
+		(fields_autoplaced yes)
+		(property "Reference" "#PWR051"
+			(at 254 59.69 0)
+			(effects
+				(font
+					(size 1.27 1.27)
+				)
+				(hide yes)
+			)
+		)
+		(property "Value" "+1V8"
+			(at 254 50.8 0)
+			(effects
+				(font
+					(size 1.27 1.27)
+				)
+			)
+		)
+		(property "Footprint" ""
+			(at 254 55.88 0)
+			(effects
+				(font
+					(size 1.27 1.27)
+				)
+				(hide yes)
+			)
+		)
+		(property "Datasheet" ""
+			(at 254 55.88 0)
+			(effects
+				(font
+					(size 1.27 1.27)
+				)
+				(hide yes)
+			)
+		)
+		(property "Description" "Power symbol creates a global label with name \"+1V8\""
+			(at 254 55.88 0)
+			(effects
+				(font
+					(size 1.27 1.27)
+				)
+				(hide yes)
+			)
+		)
+		(pin "1"
+		)
+		(instances
+			(project "simpleCarrier"
+				(path "/72db9dae-5f31-4a10-9047-fdf9bc345a06/1803d24e-9660-4c9d-82db-3dd492b14553"
+					(reference "#PWR051")
+					(unit 1)
+				)
